File: FUSH PROJECT ONE.sch (KiCad schematic (older format))
At the start: 8 parts, among them J1 AC, J2 5V, J3 LAMP, J4 ARD, K1 SRD-05VDC-SL-C, Q1 BC547

Commit message: Updated terminal labels
Parts:
- D1: symbol Diode:1N4007 -> FUSH-PROJECT-ONE-rescue:1N4007-Diode
- J1, J3: symbol Connector:Screw_Terminal_01x02 -> FUSH-PROJECT-ONE-rescue:Screw_Terminal_01x02-Connector
- J2, J4: symbol Connector:Conn_01x02_Male -> FUSH-PROJECT-ONE-rescue:Conn_01x02_Male-Connector
- K1: symbol SRD05VDC:SRD-05VDC-SL-C -> FUSH-PROJECT-ONE-rescue:SRD-05VDC-SL-C-SRD05VDC
- Q1: symbol Transistor_BJT:BC547 -> FUSH-PROJECT-ONE-rescue:BC547-Transistor_BJT
- R1: symbol Device:R_Small -> FUSH-PROJECT-ONE-rescue:R_Small-Device
Connections:
- net SIG: now reaches J4.1 (Pin_1), R1.2
- net Earth renamed GND
- net NO: no longer names the net of J3.1 (Pin_1), K1.NO
- no-connect marks 2 -> 1
Other:
- moved on the sheet: J1, J2, J3, J4, Q1, R1
Changed lines of the file:
@@
 EESchema Schematic File Version 4
+LIBS:FUSH PROJECT ONE-cache
 EELAYER 30 0
 EELAYER END
@@
 $EndDescr
 $Comp
-L Connector:Screw_Terminal_01x02 J1
+L FUSH-PROJECT-ONE-rescue:Screw_Terminal_01x02-Connector J1
 U 1 1 602E4745
-P 6650 2300
-F 0 "J1" H 6730 2292 50  0000 L CNN
-F 1 "AC" H 6730 2201 50  0000 L CNN
-F 2 "TerminalBlock:TerminalBlock_Altech_AK300-2_P5.00mm" H 6650 2300 50  0001 C CNN
-F 3 "~" H 6650 2300 50  0001 C CNN
-	1    6650 2300
-	0    -1   -1   0
-$EndComp
-$Comp
-L Device:R_Small R1
+P 7350 3400
+F 0 "J1" H 7430 3392 50  0000 L CNN
+F 1 "AC" H 7430 3301 50  0000 L CNN
+F 2 "TerminalBlock:TerminalBlock_Altech_AK300-2_P5.00mm" H 7350 3400 50  0001 C CNN
+F 3 "~" H 7350 3400 50  0001 C CNN
+	1    7350 3400
+	1    0    0    1
+$EndComp
+$Comp
+L FUSH-PROJECT-ONE-rescue:R_Small-Device R1
 U 1 1 602E8DE9
-P 2000 4550
-F 0 "R1" V 1804 4550 50  0000 C CNN
-F 1 "1K" V 1895 4550 50  0000 C CNN
-F 2 "Resistor_THT:R_Axial_DIN0207_L6.3mm_D2.5mm_P10.16mm_Horizontal" H 2000 4550 50  0001 C CNN
-F 3 "~" H 2000 4550 50  0001 C CNN
-	1    2000 4550
-	0    1    1    0
-$EndComp
-$Comp
-L Transistor_BJT:BC547 Q1
+P 4700 4450
+F 0 "R1" V 4504 4450 50  0000 C CNN
+F 1 "1K" V 4595 4450 50  0000 C CNN
+F 2 "Resistor_THT:R_Axial_DIN0207_L6.3mm_D2.5mm_P10.16mm_Horizontal" H 4700 4450 50  0001 C CNN
+F 3 "~" H 4700 4450 50  0001 C CNN
+	1    4700 4450
+	0    1    1    0
+$EndComp
+$Comp
+L FUSH-PROJECT-ONE-rescue:BC547-Transistor_BJT Q1
 U 1 1 602F1703
-P 3550 4450
-F 0 "Q1" H 3741 4496 50  0000 L CNN
-F 1 "BC547" H 3741 4405 50  0000 L CNN
-F 2 "Package_TO_SOT_THT:TO-92_Inline" H 3750 4375 50  0001 L CIN
-F 3 "http://www.fairchildsemi.com/ds/BC/BC547.pdf" H 3550 4450 50  0001 L CNN
-	1    3550 4450
-	1    0    0    -1
-$EndComp
-Wire Wire Line
-	2100 4550 3300 4550
-Wire Wire Line
-	3300 4550 3300 4450
-Wire Wire Line
-	3300 4450 3350 4450
-$Comp
-L power:Earth #PWR02
-U 1 1 602F87DB
-P 3650 5000
-F 0 "#PWR02" H 3650 4750 50  0001 C CNN
-F 1 "Earth" H 3650 4850 50  0001 C CNN
-F 2 "" H 3650 5000 50  0001 C CNN
-F 3 "~" H 3650 5000 50  0001 C CNN
-	1    3650 5000
-	1    0    0    -1
-$EndComp
-Wire Wire Line
-	3650 4650 3650 4800
-Wire Wire Line
-	3650 4250 3650 3950
-$Comp
-L power:PWR_FLAG #FLG0103
-U 1 1 6036CD49
-P 4000 4800
-F 0 "#FLG0103" H 4000 4875 50  0001 C CNN
-F 1 "PWR_FLAG" V 4000 4928 50  0000 L CNN
-F 2 "" H 4000 4800 50  0001 C CNN
-F 3 "~" H 4000 4800 50  0001 C CNN
-	1    4000 4800
-	0    1    1    0
-$EndComp
-Wire Wire Line
-	4000 4800 3650 4800
-Connection ~ 3650 4800
-Wire Wire Line
-	3650 4800 3650 4950
-$Comp
-L Connector:Conn_01x02_Male J2
+P 5300 4450
+F 0 "Q1" H 5491 4496 50  0000 L CNN
+F 1 "BC547" H 5491 4405 50  0000 L CNN
+F 2 "Package_TO_SOT_THT:TO-92_Inline" H 5500 4375 50  0001 L CIN
+F 3 "http://www.fairchildsemi.com/ds/BC/BC547.pdf" H 5300 4450 50  0001 L CNN
+	1    5300 4450
+	1    0    0    -1
+$EndComp
+$Comp
+L FUSH-PROJECT-ONE-rescue:Conn_01x02_Male-Connector J2
 U 1 1 6037200C
-P 5100 1650
-F 0 "J2" V 5162 1694 50  0000 L CNN
-F 1 "5V" V 5253 1694 50  0000 L CNN
-F 2 "Connector_PinHeader_2.54mm:PinHeader_1x02_P2.54mm_Vertical" H 5100 1650 50  0001 C CNN
-F 3 "~" H 5100 1650 50  0001 C CNN
-	1    5100 1650
-	0    1    1    0
-$EndComp
-$Comp
-L power:GND #PWR01
-U 1 1 603726C6
-P 5000 2000
-F 0 "#PWR01" H 5000 1750 50  0001 C CNN
-F 1 "GND" H 5005 1827 50  0000 C CNN
-F 2 "" H 5000 2000 50  0001 C CNN
-F 3 "" H 5000 2000 50  0001 C CNN
-	1    5000 2000
-	1    0    0    -1
-$EndComp
-Wire Wire Line
-	5000 1850 5000 1900
-Text GLabel 5100 1950 3    50   Input ~ 0
+P 1700 2500
+F 0 "J2" V 1762 2544 50  0000 L CNN
+F 1 "5V" V 1853 2544 50  0000 L CNN
+F 2 "Connector_PinHeader_2.54mm:PinHeader_1x02_P2.54mm_Vertical" H 1700 2500 50  0001 C CNN
+F 3 "~" H 1700 2500 50  0001 C CNN
+	1    1700 2500
+	0    1    1    0
+$EndComp
+Text GLabel 1850 2800 2    50   Input ~ 0
 +5V
 Wire Wire Line
-	5100 1950 5100 1850
-Text GLabel 5400 2450 1    50   Input ~ 0
-+5V
-NoConn ~ 5000 1650
-$Comp
-L SRD05VDC:SRD-05VDC-SL-C K1
+	1700 2800 1700 2700
+$Comp
+L FUSH-PROJECT-ONE-rescue:SRD-05VDC-SL-C-SRD05VDC K1
 U 1 1 6037B918
 P 6050 3100
@@
 $EndComp
 $Comp
-L Diode:1N4007 D1
+L FUSH-PROJECT-ONE-rescue:1N4007-Diode D1
 U 1 1 6035DC2B
 P 5400 3200
@@
 Wire Wire Line
 	5400 3600 5400 3350
-Wire Wire Line
-	5400 3950 5400 3600
-Wire Wire Line
-	3650 3950 5400 3950
 Connection ~ 5400 3600
 Wire Wire Line
@@
 	5400 2450 5400 2950
 Connection ~ 5400 2950
-Wire Wire Line
-	6650 2500 6650 3100
-Wire Wire Line
-	6650 3100 6350 3100
-Wire Wire Line
-	6600 3900 6350 3900
-Wire Wire Line
-	6350 3900 6350 4150
-Wire Wire Line
-	6350 4150 7200 4150
-Wire Wire Line
-	7200 4150 7200 2500
-Wire Wire Line
-	7200 2500 6750 2500
-Text GLabel 6400 3800 0    50   Input ~ 0
-NO
-$Comp
-L Connector:Screw_Terminal_01x02 J3
+$Comp
+L FUSH-PROJECT-ONE-rescue:Screw_Terminal_01x02-Connector J3
 U 1 1 6036E7A5
-P 6800 3800
-F 0 "J3" H 6880 3792 50  0000 L CNN
-F 1 "LAMP" H 6880 3701 50  0000 L CNN
-F 2 "TerminalBlock:TerminalBlock_Altech_AK300-2_P5.00mm" H 6800 3800 50  0001 C CNN
-F 3 "~" H 6800 3800 50  0001 C CNN
-	1    6800 3800
-	1    0    0    -1
-$EndComp
-Wire Wire Line
-	6400 3800 6600 3800
-Text GLabel 6450 3000 2    50   Input ~ 0
-NO
+P 7350 2950
+F 0 "J3" H 7430 2942 50  0000 L CNN
+F 1 "LAMP" H 7430 2851 50  0000 L CNN
+F 2 "TerminalBlock:TerminalBlock_Altech_AK300-2_P5.00mm" H 7350 2950 50  0001 C CNN
+F 3 "~" H 7350 2950 50  0001 C CNN
+	1    7350 2950
+	1    0    0    -1
+$EndComp
 Wire Wire Line
 	6350 3000 6450 3000
 NoConn ~ 6350 3300
-Text GLabel 4900 1900 0    50   Input ~ 0
--5V
-Wire Wire Line
-	4900 1900 5000 1900
-Connection ~ 5000 1900
-Wire Wire Line
-	5000 1900 5000 2000
-Text GLabel 3550 4950 0    50   Input ~ 0
--5V
-Wire Wire Line
-	3550 4950 3650 4950
-Connection ~ 3650 4950
-Wire Wire Line
-	3650 4950 3650 5000
-$Comp
-L Connector:Conn_01x02_Male J4
+Text GLabel 1500 2800 0    50   Input ~ 0
+GND
+Wire Wire Line
+	1500 2800 1600 2800
+$Comp
+L FUSH-PROJECT-ONE-rescue:Conn_01x02_Male-Connector J4
 U 1 1 60362F2F
-P 1350 4550
-F 0 "J4" V 1412 4594 50  0000 L CNN
-F 1 "ARD" V 1503 4594 50  0000 L CNN
-F 2 "Connector_PinHeader_2.54mm:PinHeader_1x02_P2.54mm_Vertical" H 1350 4550 50  0001 C CNN
-F 3 "~" H 1350 4550 50  0001 C CNN
-	1    1350 4550
-	1    0    0    -1
-$EndComp
-Wire Wire Line
-	1550 4550 1900 4550
-Text GLabel 1750 4750 3    50   Input ~ 0
--5V
-Wire Wire Line
-	1750 4650 1750 4750
-Wire Wire Line
-	1550 4650 1750 4650
+P 1700 3850
+F 0 "J4" V 1762 3894 50  0000 L CNN
+F 1 "ARD" V 1853 3894 50  0000 L CNN
+F 2 "Connector_PinHeader_2.54mm:PinHeader_1x02_P2.54mm_Vertical" H 1700 3850 50  0001 C CNN
+F 3 "~" H 1700 3850 50  0001 C CNN
+	1    1700 3850
+	0    1    1    0
+$EndComp
+Text GLabel 1450 4250 0    50   Input ~ 0
+GND
+Wire Wire Line
+	1850 2800 1700 2800
+Wire Wire Line
+	6350 3100 6600 3100
+Wire Wire Line
+	6600 3100 6600 3400
+Wire Wire Line
+	6600 3400 7150 3400
+Wire Wire Line
+	7150 3300 7000 3300
+Wire Wire Line
+	7000 3300 7000 3050
+Wire Wire Line
+	7000 3050 7150 3050
+Wire Wire Line
+	7150 2950 6450 2950
+Wire Wire Line
+	6450 2950 6450 3000
+Wire Wire Line
+	4800 4450 5100 4450
+Wire Wire Line
+	5400 3600 5400 4250
+Wire Wire Line
+	1450 4250 1600 4250
+Wire Wire Line
+	1600 4250 1600 4050
+Text GLabel 1850 4250 2    50   Input ~ 0
+SIG
+Wire Wire Line
+	1850 4250 1700 4250
+Wire Wire Line
+	1700 4050 1700 4250
+Wire Wire Line
+	1600 2700 1600 2800
+Text GLabel 4350 4450 0    50   Input ~ 0
+SIG
+Wire Wire Line
+	4350 4450 4600 4450
+Text GLabel 1450 5450 0    50   Input ~ 0
+GND
+$Comp
+L FUSH-PROJECT-ONE-rescue:GND-power #PWR?
+U 1 1 625CB80F
+P 1700 5700
+F 0 "#PWR?" H 1700 5450 50  0001 C CNN
+F 1 "GND-power" H 1705 5527 50  0000 C CNN
+F 2 "" H 1700 5700 50  0001 C CNN
+F 3 "" H 1700 5700 50  0001 C CNN
+	1    1700 5700
+	1    0    0    -1
+$EndComp
+Wire Wire Line
+	1700 5700 1700 5450
+Wire Wire Line
+	1700 5450 1450 5450
+$Comp
+L FUSH-PROJECT-ONE-rescue:GND-power #PWR?
+U 1 1 625CD3EF
+P 5400 5150
+F 0 "#PWR?" H 5400 4900 50  0001 C CNN
+F 1 "GND-power" H 5405 4977 50  0000 C CNN
+F 2 "" H 5400 5150 50  0001 C CNN
+F 3 "" H 5400 5150 50  0001 C CNN
+	1    5400 5150
+	1    0    0    -1
+$EndComp
+Text GLabel 5400 2450 1    50   Input ~ 0
++5V
+Wire Wire Line
+	5400 5150 5400 4800
+Wire Wire Line
+	5400 4650 5400 4800
+Connection ~ 5400 4800
+Wire Wire Line
+	5750 4800 5400 4800
+$Comp
+L FUSH-PROJECT-ONE-rescue:PWR_FLAG-power #FLG0103
+U 1 1 6036CD49
+P 5750 4800
+F 0 "#FLG0103" H 5750 4875 50  0001 C CNN
+F 1 "PWR_FLAG-power" V 5750 4928 50  0000 L CNN
+F 2 "" H 5750 4800 50  0001 C CNN
+F 3 "~" H 5750 4800 50  0001 C CNN
+	1    5750 4800
+	0    1    1    0
+$EndComp
 $EndSCHEMATC
